File: hardware/TEG.kicad_pcb (KiCad board)
At the start: 2 copper layers, 107.7 x 84.4 mm, 30 parts, among them J1 TEG_IN, J2 FAN_4PIN, J3 TEST_LOAD, Q1 AO3400A, U1 BQ25504RGTT, U2 MT3608

Commit message: Add MPPT sampling network; switch storage to supercapacitor
The BQ25504 has MPPT built in, but the draft was missing its sampling
network. Fixed:

- Add R13/R14 = 10M/10M on VOC_SAMP -> MPP ratio ~50% of Voc
  (TEG matched load; the datasheet's 78% default targets solar)
- CREF/CBYP = 10nF (C1589); drop the 100nF cap that would have slowed
  the high-impedance sampling node
- Fix OV/UV chain order to the datasheet topology and add the missing
  third OK-chain resistor (R15); set threshold values from the datasheet
  worked example (VBAT_OV 3.15V / UV 2.20V / OK 2.44V / HYST 2.80V)
- R5 = 0R ties OT_PROG to GND (65C charge cutoff)
- L1/L2 corrected to the datasheet-recommended 22uH

Storage = supercapacitor 0.22-0.47F/5.5V instead of a battery: safer in a
thermal device (no fire/cold-plating risk), simpler, matches the fan's
burst load. Trade-off noted: measure leakage vs harvest current.

32 parts / 85 pins. ERC: 1 intentional warning; board DRC: 0 violations.
BOM rev B; several high-ohm 1% resistors, the 22uH inductor and the
supercap still need JLCPCB part numbers (all extended / hand-solder).

Co-authored-by: Copilot <223556219+Copilot@users.noreply.github.com>
Parts:
- removed C2: 100nF, TEG:C0603
- added R13: 10M, TEG:R0603, F.Cu at (46.0, 44.0)
- added R14: 10M, TEG:R0603, F.Cu at (46.0, 50.0)
- added R15: 4.42M, TEG:R0603, F.Cu at (22.0, 76.0)
- C3, C8: value 100nF -> 10nF
- L1, L2: value 4.7uH -> 22uH
- R1: value TBD -> 5.90M
- R2: value TBD -> 4.02M
- R3: value TBD -> 5.60M
- R4: value TBD -> 4.42M
- R5: value TBD -> 0R
- R6: value TBD -> 1.43M
- R7: value TBD -> 4.22M
Connections:
- R1 pad 2: VRDIV -> VBAT_OV
- R2 pad 1: VRDIV -> VBAT_OV
- R2 pad 2: VBAT_OV -> VRDIV
- R3 pad 1: VBAT_OV -> VRDIV

Commit message: Source every part from the JLCPCB catalogue; document the storage decision
jlc-client's search index degraded to returning the same high-stock list
for every query, so add scripts/jlc_lookup.py which queries JLCPCB's own
parts API and reports id + library type + stock.

All 31 machine-placed parts now verified in the catalogue:
- 22uH inductor -> C82401 (SWPA4020S220MT, 4x4mm, 1.05A)
- odd E96 threshold resistors -> C2076902/C137708/C23190/C166806/
  C166807/C166898 (all in stock)
- MT3608 divider computed: 73.2k/10k -> 5.0V (C2933257/C25804)
- R10 -> 1k base part C21190
Flag: BQ25504RGTT (C157471) is low stock (7); C2876746 is the same part.

Confirmed via JLCPCB's API that supercapacitors and batteries are not
stocked at all (0 results), so BOM.md now lays out four storage options
(hand-solder supercap / plug-in header / coin-cell holder / electrolytic)
with stored energy and effort for each.

Normalise pin electrical types in the symbol library (not just at embed
time) and embed library text verbatim, removing the power-pin ERC errors.

ERC: 1 intentional + 2 cosmetic warnings; board DRC: 0 violations.

Co-authored-by: Copilot <223556219+Copilot@users.noreply.github.com>
Parts:
- L1, L2: footprint TEG:IND-SMD_L2.5-W2.0-VLS252012CX-150M -> TEG:IND-SMD_L4.0-W4.0
- R8: value TBD -> 73.2k
- R9: value TBD -> 10k

Commit message: Storage: option D electrolytic buffer (100% JLCPCB assembled)
The user chose the fully-automated path: no supercap, no battery. Adds
C2 = 1000uF 6.3V SMD electrolytic (C970711) as the VBAT buffer, which is
what the BQ25504 needs to operate (datasheet reference shows >100uF).

Consequences documented rather than glossed over: with ~5mJ stored (vs
~1.2J for a supercap) the fan can only run on live harvest, not from
storage. VBAT_OK is left unconnected with a no-connect marker; the
datasheet confirms it is a low-drive digital output referenced to VSTOR,
so gating the load would need extra parts - deferred.

Also: pin-type normalisation now never clobbers power pins (a previous
pass had turned PWR_FLAG's power_out into passive, which made 4 power
nets report as undriven).

Board = 33 parts. ERC: 3 cosmetic warnings. DRC: 1 cosmetic silkscreen
warning. Remaining: routing.

Co-authored-by: Copilot <223556219+Copilot@users.noreply.github.com>
Parts:
- added C2: 1000uF, TEG:CAP-SMD_BD8.0-L8.3-W8.3-LS9.3-FD-1, F.Cu at (60.0, 48.0)
Connections:
- U1 pad 11: VBAT_OK -> (no net)

Commit message: Route the board with FreeRouting: DRC-clean, fab outputs generated
KiCad has no autorouter, so this uses the standard SPECCTRA round-trip,
scripted in scripts/freeroute.sh:
  pcbnew ExportSpecctraDSN -> freerouting -de/-do -> ImportSpecctraSES -> DRC

FreeRouting reported 0 unrouted and 0 violations on both the routing and
optimisation passes, and KiCad's DRC agrees: 0 violations, 0 unconnected
items. It does the rip-up-and-retry the hand-written route_board.py
lacked.

Details:
- Net classes (Default, Power) are defined in gen_board.py and exported
  into the DSN so the router obeys them. Widths are 0.2mm for both: the
  power/GND nets also land on U1's 0.5mm-pitch pins where a wider track
  cannot escape, and the autorouter will not taper.
- Needed a JDK 25 for the FreeRouting jar - the bundled native CLI build
  crashes with a GraalVM serialization error.
- Lowered the board minimum track width to 0.15mm (above JLCPCB's 0.127
  floor) because FreeRouting fans out U1 at 0.15mm.
- Moved C2's reference text in the footprint so it clears its own
  silkscreen: DRC now reports zero violations.

Fabrication outputs in build/fab/ (gitignored): gerbers, Excellon drill,
position file, JLCPCB-format BOM, and review PDFs.

Co-authored-by: Copilot <223556219+Copilot@users.noreply.github.com>
Routing:
- net GND: track 0.00 -> 278.3 mm, vias 0 -> 7
- net VBAT: track 0.00 -> 123.7 mm, vias 0 -> 4
- net +5V: track 0.00 -> 88.0 mm, vias 0 -> 1
- net OK_PROG: track 0.00 -> 75.7 mm, vias 0 -> 2
- net TEG+: track 0.00 -> 70.1 mm, vias 0 -> 3
- net OK_HYST: track 0.00 -> 70.1 mm, vias 0 -> 2
- net VSTOR: track 0.00 -> 66.1 mm
- net OT_PROG: track 0.00 -> 48.3 mm, vias 0 -> 2
- net FAN_PWM: track 0.00 -> 47.4 mm, vias 0 -> 1
- net VOC_SAMP: track 0.00 -> 45.8 mm, vias 0 -> 2
- net VBAT_UV: track 0.00 -> 43.2 mm
- net VRDIV: track 0.00 -> 35.7 mm
- net VBAT_OV: track 0.00 -> 30.7 mm
- net FB_5V: track 0.00 -> 26.9 mm, vias 0 -> 2
- net VREF_SAMP: track 0.00 -> 22.0 mm, vias 0 -> 2
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